File: hardware/bt-mp3/bt-mp3.kicad_sch (KiCad schematic)
At the start: 12 parts, among them J1 USB_C_Receptacle_USB2.0_16P, J2 BATT, U1 SF32LB527UD6, Y1 48M

Commit message: add: 基础的外围器件
Parts:
- removed AE1: Antenna, symbol Device:Antenna
- added AE1: 蓝牙天线, chenxuuu_Module:bt_ant, symbol Device:Antenna_Shield
- added C10: 4.7uF/10V, symbol Device:C
- added C11, C12, C19: 1uF, symbol Device:C
- added C13, C14, C15, C5: 4.7uF, symbol Device:C
- added C16: 0.47uF, symbol Device:C
- added C17: 0.1uF, symbol Device:C
- added C18, C6, C7, C8: 2.2uF/10V, symbol Device:C
- added C9: NF, symbol Device:C
- added D1: RED, LED_SMD:LED_0402_1005Metric, symbol Device:LED
- added D2: GREEN, LED_SMD:LED_0402_1005Metric, symbol Device:LED
- added D3: ESD5311N-2, Diode_THT:D_DO-201AE_P15.24mm_Horizontal, symbol Diode:1N630xCA
- added J3: LCD, chenxuuu_Module:1.47LCD-IPS-172x320-font, symbol Connector_Generic:Conn_01x12
- added L1: 4.7uH, Inductor_SMD:L_Murata_DFE201610P, symbol Device:L
- added Q1: SS8050, Package_TO_SOT_SMD:SOT-23, symbol Transistor_BJT:SS8050
- added R10: 100K, symbol Device:R
- added R4, R5: 1K, Resistor_SMD:R_0402_1005Metric, symbol Device:R
- added R6: 10K, symbol Device:R
- added R7, R9: 5.1K, symbol Device:R
- added R8: 10R, symbol Device:R
- added SW1: Side_SWITCH_SW_3*6*3.5mm, chenxuuu_Module:3x6x3.5_SW_side, symbol chenxuuu_Library:Side_SWITCH_SW_3*6*3.5mm
- added SW2: SW_SPST, chenxuuu_Module:MSK-0002, symbol Switch:SW_SPST
- added TPG, TPR, TPT: TestPoint, TestPoint:TestPoint_Pad_D1.5mm, symbol Connector:TestPoint
- added U2: PY25Q128HA-WXH-IR, Package_SO:SOIC-8_5.23x5.23mm_P1.27mm, symbol Memory_Flash:W25Q128JVP
- U1: symbol btlib:SF32LB52xUx -> chenxuuu_Library:SF32LB52xUx
Connections:
- net +BATT: now also SW2.1 (A); no longer C2.1, U1.24 (VCC)
- net GND: now also C1.1, C2.1, AE1.2 (Shield), C10.2, C11.2, C12.2, C13.2, C14.2, C15.2, C16.2, C17.2, C18.2, C19.2, C5.2, C6.2, C7.2, C8.2, C9.2, D1.1 (K), D2.1 (K), D3.1 (A1), J3.1 (Pin_1), J3.12 (Pin_12), J3.5 (Pin_5), J3.6 (Pin_6), Q1.2 (E), R10.1, R6.1, SW1.3, TPG.1, U2.4 (GND); no longer C1.2, C2.2
- net USB_DM: now also U1.64 (PA36)
- net USB_DP: now also U1.65 (PA35)
- net VBUS: now also C1.2; no longer C1.1
- net at C4.1, R3.1: now also AE1.1 (A)
- net at U1.12 (VDD_RTC): now also C12.1
- net at U1.13 (VDD_RET): now also C16.1
- net VDD33_VOUT2: now reaches U1.14 (VDD33_VOUT2)
- net VDD33_VOUT2: now also C8.1, J3.3 (Pin_3)
- net at U1.15 (VDD_VOUT2): now also C15.1
- net at U1.16 (VDD_VOUT1): now also C13.1
- net at U1.17 (BUCK_FB): now also C10.1, L1.2
- net at U1.18 (BUCK_LX): now also C9.1, L1.1
- net VSYS: now reaches U1.19 (VSYS)
- net VSYS: now also U1.52 (AVDD_BRF), C5.1, C6.1, R7.1
- net VDD33_VOUT1: now reaches U1.22 (VDD33_VOUT1)
- net VDD33_VOUT1: now also U1.38 (AVDD33_AUD), C17.1, C18.1, C7.1, J3.4 (Pin_4), U2.8 (VCC)
- net at U1.23 (VDD18_VOUT): now also C11.1
- net at U1.68 (GPADC_VREF): now also C14.1
- net DBG_TX: now reaches U1.26 (PA19)
- net DBG_TX: now also TPT.1
- net DBG_RX: now reaches U1.27 (PA18)
- net DBG_RX: now also TPR.1
- net PA_17_MPI2_D3: now reaches U1.28 (PA17)
- net PA_17_MPI2_D3: now also U2.7 (IO3)
- net PA_16_MPI2_CLK: now reaches U1.29 (PA16)
- net PA_16_MPI2_CLK: now also U2.6 (CLK)
- net PA_15_MPI2_D0: now reaches U1.30 (PA15)
- net PA_15_MPI2_D0: now also U2.5 (DI(IO0))
- net PA_14_MPI2_D2: now reaches U1.31 (PA14)
- net PA_14_MPI2_D2: now also U2.3 (IO2)
- net PA_13_MPI2_D1: now reaches U1.32 (PA13)
- net PA_13_MPI2_D1: now also U2.2 (DO(IO1))
- net PA_12_MPI2_CS: now reaches U1.33 (PA12)
- net PA_12_MPI2_CS: now also U2.1 (~{CS})
- net DAC_N: now reaches U1.36 (DACN)
- net DAC_P: now reaches U1.37 (DACP)
- net at U1.39 (AUD_VREF): now also C19.1
- net PA06_LCD_DC: now reaches U1.45 (PA6)
- net PA06_LCD_DC: now also J3.7 (Pin_7)
- net PA05_LCD_DAT: now reaches U1.46 (PA5)
- net PA05_LCD_DAT: now also J3.10 (Pin_10)
- net PA04_LCD_SCL: now reaches U1.47 (PA4)
- net PA04_LCD_SCL: now also J3.9 (Pin_9)
- net PA03_LCD_CS: now reaches U1.48 (PA3)
- net PA03_LCD_CS: now also J3.8 (Pin_8)
- net LCD_LED_PWM: now reaches U1.50 (PA1)
- net LCD_LED_PWM: now also R9.1
- net PA00_LCD_RESET: now reaches U1.51 (PA0)
- net PA00_LCD_RESET: now also J3.11 (Pin_11)
- net PA34_POWER_KEY: now reaches U1.66 (PA34)
- net PA34_POWER_KEY: now also D3.2 (A2), R6.2, SW1.1
- new net: C2.2, SW2.2 (B), U1.24 (VCC)
- new net: J3.2 (Pin_2), R8.2
- new net: Q1.1 (B), R10.2, R9.2
- new net: R7.2, SW1.2
- new net: Q1.3 (C), R8.1
- new net: D2.2 (A), R5.2
- new net: D1.2 (A), R4.2
- new net GREEN_LED: R5.1
- new net RED_LED: R4.1
Other:
- note added: "PWM调背光"
- note added: "USB口"
- note added: "充电状态灯"
- note added: "外接FLASH"
- note added: "屏幕"
- note added: "开机键"
- note added: "调试下载"
- moved on the sheet: C1, C3, C4, J1, R1, R2, R3, U1B, Y1

Commit message: update: 完成原理图
Parts:
- removed C18: 2.2uF/10V, symbol Device:C
- removed C19: 1uF, symbol Device:C
- removed R5: 1K, Resistor_SMD:R_0402_1005Metric, symbol Device:R
- removed TPR, TPT: TestPoint, TestPoint:TestPoint_Pad_D1.5mm, symbol Connector:TestPoint
- added C20: 0.1uF, symbol Device:C
- added J4: TF-021B-H265, chenxuuu_Module:TF-SMD_TF-021B-H265, symbol chenxuuu_Library:TF-021B-H265
- added Q2: SS8050, Package_TO_SOT_SMD:SOT-23, symbol Transistor_BJT:SS8050
- added R11: 1M, Resistor_SMD:R_0402_1005Metric, symbol Device:R
- added R12: 2M, Resistor_SMD:R_0402_1005Metric, symbol Device:R
- added R13, R14, R15, R16, R22: 100K, symbol Device:R
- added R21: 5.1K, symbol Device:R
- added R23: 1K, symbol Device:R
- added SW3, SW4: Side_SWITCH_SW_3*6*3.5mm, chenxuuu_Module:3x6x3.5_SW_side, symbol chenxuuu_Library:Side_SWITCH_SW_3*6*3.5mm
- added SW5: ~, chenxuuu_Module:SIQ-02FVS3_1, symbol chenxuuu_Library:SIQ-02FVS3
- added TP2, TP3, TP4, TP5, TP6, TP7: TestPoint, TestPoint:TestPoint_Pad_D1.5mm, symbol Connector:TestPoint
- added Y2: 32.768KHz/7pF, Crystal:Crystal_SMD_3215-2Pin_3.2x1.5mm, symbol Device:Crystal
- D2: value GREEN -> WHITE
- D3: footprint Diode_THT:D_DO-201AE_P15.24mm_Horizontal -> chenxuuu_Module:DFN1006-2_L1.0-W0.6-RD
- renumbered TPG to TP1
Connections:
- net RED_LED is gone; now on net VBUS: R4.1
- net +BATT: now also R11.1, TP5.1
- net DBG_RX: now also TP3.1
- net DBG_TX: now also TP2.1
- net GND: now also C20.2, J4.10 (SHIELD), J4.6 (VSS), J4.9 (SHIELD), Q2.2 (E), R12.2, R22.1, SW3.3, SW4.3, SW5.1 (EH), SW5.2 (EH), SW5.3 (EH), SW5.4 (EH), SW5.5 (EH), SW5.6 (EH), SW5.C; no longer D2.1 (K)
- net VDD33_VOUT1: now also D2.2 (A), J3.3 (Pin_3), TP7.1; no longer U1.38 (AVDD33_AUD)
- net VDD33_VOUT2: now also J4.4 (VDD), R13.2, R14.2, R15.2, R16.2, TP6.1; no longer J3.3 (Pin_3)
- net VSYS: now also SW3.2, SW4.2, TP4.1
- net KEY1: now reaches U1.1 (PA32)
- net KEY1: now also SW3.1
- net at U1.10 (PA23): now also Y2.2
- net at U1.11 (PA22): now also Y2.1
- net BAT_ADC: now reaches U1.2 (PA31)
- net BAT_ADC: now also C20.1, R11.2, R12.1
- net WHITE_LED: now reaches U1.25 (PA20)
- net WHITE_LED: now also R21.1
- net TF_SPI_CS: now reaches U1.4 (PA29)
- net TF_SPI_CS: now also J4.2 (DAT3/CD), R13.1
- net KEYB: now reaches U1.42 (PA9)
- net KEYB: now also SW5.B
- net KEYA: now reaches U1.43 (PA8)
- net KEYA: now also SW5.A
- net KEY3: now reaches U1.44 (PA7)
- net KEY3: now also SW5.S
- net TF_SPI_CLK: now reaches U1.5 (PA28)
- net TF_SPI_CLK: now also J4.5 (CLK), R15.1
- net KEY2: now reaches U1.67 (PA33)
- net KEY2: now also SW4.1
- net TF_SPI_MISO: now reaches U1.8 (PA25)
- net TF_SPI_MISO: now also J4.7 (DAT0), R16.1
- net TF_SPI_MOSI: now reaches U1.9 (PA24)
- net TF_SPI_MOSI: now also J4.3 (CMD), R14.1
- net DAC_N: no longer names the net of U1.36 (DACN)
- net DAC_P: no longer names the net of U1.37 (DACP)
- new net: Q2.1 (B), R21.2, R22.2
- new net: Q2.3 (C), R23.1
- new net: D2.1 (K), R23.2
- no-connect marks 2 -> 24
Other:
- note added: "USB指示灯"
- note added: "主FLASH"
- note added: "充电状态灯 呼吸灯"
- note added: "按键1"
- note added: "按键2"
- note added: "旋转编码器+按键"
- note added: "电池电压检测"
- note added: "电源检查"
- note removed: "充电状态灯"
- note removed: "外接FLASH"
- moved on the sheet: D1, D2, D3, R4, R6, R7, SW1, TP1

Commit message: add: 原理图信息
Other:
- company: (none) -> chenxuuu
- title: (none) -> BT MP3 蓝牙MP3小板
Changed lines of the file:
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@@
 	(generator_version "8.0")
 	(paper "A4")
+	(title_block
+		(title "BT MP3 蓝牙MP3小板")
+		(date "2025-02-06")
+		(rev "001")
+		(company "chenxuuu")
+	)
 	(junction
 		(at 133.35 64.77)

Commit message: update: 分配好封装
Parts:
- removed SW2: SW_SPST, chenxuuu_Module:MSK-0002, symbol Switch:SW_SPST
- added SW6: SS-22F25-G050, chenxuuu_Module:MS-22C01-G010, symbol chenxuuu_Library:SS-22F25-G050
- C1, C10, C11, C12, C13, C14, C15, C16, C17, C2, C20, C3, C4, C5, C6, C7, C8, C9: footprint (none) -> Capacitor_SMD:C_0402_1005Metric
- J2: footprint Connector_AMASS:AMASS_XT30PW-F_1x02_P2.50mm_Horizontal -> TerminalBlock_Phoenix:TerminalBlock_Phoenix_PTSM-0,5-2-HV-2.5-SMD_1x02-1MP_P2.50mm_Vertical
- R1, R10, R13, R14, R15, R16, R2, R21, R22, R23, R3, R6, R7, R8, R9: footprint (none) -> Resistor_SMD:R_0402_1005Metric
Connections:
- net +BATT: now also SW6.1, SW6.4
- net at C2.2, U1.24 (VCC): now also SW6.2, SW6.5
- no-connect marks 24 -> 26

Commit message: add: 布线
Parts:
- removed TP5: TestPoint, TestPoint:TestPoint_Pad_D1.5mm, symbol Connector:TestPoint
- added C18: 0.1uF, Capacitor_SMD:C_0402_1005Metric, symbol Device:C
- AE1: footprint chenxuuu_Module:bt_ant -> chenxuuu_Module:bt_ant_mirror
- J1: footprint Connector_USB:USB_C_Receptacle_G-Switch_GT-USB-7010ASV -> Connector_USB:USB_C_Receptacle_GCT_USB4105-xx-A_16P_TopMnt_Horizontal
- J2: footprint TerminalBlock_Phoenix:TerminalBlock_Phoenix_PTSM-0,5-2-HV-2.5-SMD_1x02-1MP_P2.50mm_Vertical -> Connector_Hirose:Hirose_DF13C_CL535-0402-2-51_1x02-1MP_P1.25mm_Vertical
Connections:
- net GND: now also SW3.2, SW4.2, C18.2
- net KEY1: now also U1.44 (PA7); no longer U1.1 (PA32)
- net KEY2: now also U1.49 (PA2); no longer U1.67 (PA33)
- net KEY3: now also U1.42 (PA9); no longer U1.44 (PA7)
- net KEYB: now also U1.35 (PA10); no longer U1.42 (PA9)
- net VDD33_VOUT2: now also C18.1
- net VSYS: no longer SW3.2, SW4.2
- net WHITE_LED: now also U1.34 (PA11); no longer U1.25 (PA20)
- no-connect marks 26 -> 25
